File: afterglow_gi_nano/afterglow_gi_nano.kicad_pcb (KiCad board)
At the start: 2 copper layers, 195 x 125 mm, 53 parts, among them J1 Conn_02x17_Odd_Even, J2 POWER_CONN, J3 GI_WPC_J120, J4 GI_WPC_J121, J5 GI_CONN_J119, J6 Conn_02x17_Odd_Even, Q1 FQP30N06L, Q2 FQP30N06L, Q3 FQP30N06L, Q4 FQP30N06L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

Commit message: Designing the PCB
Parts:
- removed J6: Conn_02x17_Odd_Even, Pin_Headers:Pin_Header_Straight_2x17_Pitch2.54mm
- J2: footprint Connectors_Molex:Molex_KK-41791-02_02x3.96mm_Straight -> Connectors_Terminal_Blocks:TerminalBlock_Philmore_TB132_02x5mm_Straight
- U1: footprint Housings_DIP:DIP-20_W7.62mm_LongPads -> Housings_SOIC:SOIC-20W_7.5x12.8mm_Pitch1.27mm
- moved Q1 270.2 mm to (63.0, 73.5), turned to 270 degrees
- moved C1 223.5 mm to (16.5, 43.2)
- moved C2 223.5 mm to (21.1, 43.2)
- moved Q2 223.2 mm to (71.5, 73.5), turned to 270 degrees
- moved Q3 219.4 mm to (79.5, 73.5), turned to 270 degrees
- moved R3 211.5 mm to (47.6, 38.0)
- moved R1 168.7 mm to (43.9, 57.1)
- moved R15 168.7 mm to (39.1, 57.1)
- moved C3 157.2 mm to (34.9, 74.9)
- moved R10 157.2 mm to (39.6, 85.9)
- moved R11 157.2 mm to (39.6, 87.8)
- moved R12 157.2 mm to (33.0, 129.5)
- moved R13 157.2 mm to (37.0, 94.9)
- moved R14 157.2 mm to (30.2, 74.9)
- moved R16 157.2 mm to (37.0, 96.8)
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Connections:
- C2 pad 1: +12V -> Net-(C2-Pad1)
- D6 pad 1: +12V -> Net-(C2-Pad1)
- D6 pad 2: Net-(D6-Pad2) -> +12V
- J2 pad 2: Net-(D6-Pad2) -> +12V
- U2 pad 1: +12V -> Net-(C2-Pad1)
Routing:
- net /GI_OUT_4: track 0.00 -> 47.1 mm
- net Net-(F1-Pad1): track 0.00 -> 37.1 mm
- net Net-(F5-Pad1): track 0.00 -> 13.0 mm
- net Net-(F4-Pad1): track 0.00 -> 13.0 mm
- net Net-(F3-Pad1): track 0.00 -> 13.0 mm
- net Net-(F2-Pad1): track 0.00 -> 13.0 mm
- net /GI_OUT_3: track 0.00 -> 13.0 mm
- net /GI_OUT_2: track 0.00 -> 13.0 mm
- net /GI_OUT_1: track 0.00 -> 13.0 mm
- net /GI_OUT_0: track 0.00 -> 13.0 mm
Other:
- board outline removed
- net class 12V added: clearance 0.5, trace_width 1.75, via_dia 2, via_drill 1

Commit message: Some PCB progress
Parts:
- moved D2 108.4 mm to (110.7, 107.0), turned to 0 degrees
- moved D1 102.2 mm to (110.7, 102.5), turned to 0 degrees
- moved R24 98.3 mm to (87.7, 45.0)
- moved R7 97.4 mm to (99.0, 78.3), turned to 90 degrees
- moved D5 96.3 mm to (110.7, 98.0), turned to 0 degrees
- moved R4 95.8 mm to (99.0, 70.3), turned to 90 degrees
- moved D3 90.4 mm to (110.7, 93.5), turned to 0 degrees
- moved R23 86.3 mm to (86.7, 41.0)
- moved D4 84.8 mm to (110.7, 89.0), turned to 0 degrees
- moved R3 76.0 mm to (46.4, 114.0)
- moved R17 75.6 mm to (102.0, 105.3), turned to 90 degrees
- moved R14 74.9 mm to (102.0, 96.3), turned to 90 degrees
- moved R5 63.5 mm to (102.0, 70.3), turned to 90 degrees
- moved R2 63.3 mm to (83.0, 43.6), turned to 90 degrees
- moved R8 62.7 mm to (102.0, 78.3), turned to 90 degrees
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Routing:
- net +12V: track 0.00 -> 74.0 mm
- net GND: track 0.00 -> 55.3 mm
- net /ZC: track 0.00 -> 40.8 mm
- net /D7: track 0.00 -> 37.4 mm
- net /D6: track 0.00 -> 29.8 mm, vias 0 -> 1
- net /TRIAC: track 0.00 -> 23.1 mm, vias 0 -> 1
- net /D3: track 0.00 -> 23.0 mm, vias 0 -> 1
- net /D1: track 0.00 -> 23.0 mm, vias 0 -> 1
- net /BLANK: track 0.00 -> 22.4 mm, vias 0 -> 1
- net /D2: track 0.00 -> 22.4 mm, vias 0 -> 1
- net /D0: track 0.00 -> 22.4 mm, vias 0 -> 1
- net /D5: track 0.00 -> 20.1 mm, vias 0 -> 1
- net /D4: track 0.00 -> 16.7 mm, vias 0 -> 1
Other:
- board outline added: 64 x 110 mm
- net class Default: clearance 0.2 -> 0.25; trace_width 0.25 -> 0.3
- rule trace_clearance: 0.2 -> 0.25

Commit message: Some PCB progress
Parts:
- R10, R11, R12, R13, R14, R15, R16, R17, R3, R4, R5, R6, R7, R8, R9: moved to B.Cu
- moved R20 92.8 mm to (116.7, 94.0)
- moved R19 92.4 mm to (117.3, 107.0)
- moved R21 86.6 mm to (116.7, 89.0)
- moved R15 79.6 mm to (79.0, 126.0), turned to 270 degrees
- moved R22 73.2 mm to (117.3, 98.0)
- moved R18 70.0 mm to (117.0, 103.0)
- moved C3 66.6 mm to (88.0, 34.8), turned to 90 degrees
- moved R16 53.1 mm to (58.5, 71.0), turned to 270 degrees
- moved R17 53.1 mm to (61.5, 71.0), turned to 270 degrees
- moved R7 45.0 mm to (58.5, 98.0), turned to 270 degrees
- moved R8 45.0 mm to (61.5, 98.0), turned to 270 degrees
- moved R10 44.6 mm to (58.5, 106.0), turned to 270 degrees
- moved R11 44.6 mm to (61.5, 106.0), turned to 270 degrees
- moved R4 44.6 mm to (58.5, 89.0), turned to 270 degrees
- moved R5 44.6 mm to (61.5, 89.0), turned to 270 degrees
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Routing:
- net GND: track 55.3 -> 209.6 mm
- net Net-(F1-Pad1): track 37.1 -> 96.4 mm
- net /GI_OUT_4: track 47.1 -> 100.4 mm
- net +12V: track 74.0 -> 124.6 mm
- net Net-(F2-Pad1): track 13.0 -> 61.0 mm
- net /GI_OUT_3: track 13.0 -> 55.6 mm
- net /GI_OUT_0: track 13.0 -> 50.9 mm
- net Net-(F3-Pad1): track 13.0 -> 50.4 mm
- net Net-(F4-Pad1): track 13.0 -> 39.2 mm
- net /GI_OUT_1: track 13.0 -> 37.2 mm
- net Net-(F5-Pad1): track 13.0 -> 27.6 mm
- net /GI_OUT_2: track 13.0 -> 27.1 mm
Other:
- net class Default: clearance 0.25 -> 0.5; trace_width 0.3 -> 1.75
- rule trace_clearance: 0.25 -> 0.5

Commit message: Some PCB progress
Parts:
- moved R19 15.4 mm to (113.7, 92.0), turned to 180 degrees
- moved R18 15.4 mm to (113.7, 88.0), turned to 180 degrees
- moved D2 15.4 mm to (107.3, 92.0)
- moved D1 14.9 mm to (107.3, 88.0)
- moved D4 11.5 mm to (107.3, 100.0)
- moved R21 11.4 mm to (113.7, 100.0), turned to 180 degrees
- moved R22 7.05 mm to (113.7, 104.0), turned to 180 degrees
- moved D5 6.85 mm to (107.3, 104.0)
- moved D3 4.14 mm to (107.3, 96.0)
- moved R20 3.61 mm to (113.7, 96.0), turned to 180 degrees
- moved J2 3.54 mm to (109.5, 121.5)
- moved R4 1.03 mm to (57.5, 88.8)
- moved R5 1.03 mm to (60.5, 88.8)
Routing:
- net Net-(C2-Pad1): track 0.00 -> 23.1 mm
- net /5V: track 0.00 -> 6.75 mm
- net Net-(F1-Pad1): track 96.4 -> 90.1 mm
- net GND: track 209.6 -> 213.5 mm
- net +12V: track 124.6 -> 127.3 mm
- net /GI_OUT_4: track 100.4 -> 98.3 mm
- net /GI_OUT_0: track 50.9 -> 51.6 mm
Other:
- net class 12V: clearance 0.5 -> 0.3; trace_width 1.75 -> 0.5
- net class Default: clearance 0.5 -> 0.3; trace_width 1.75 -> 0.5
- rule trace_clearance: 0.5 -> 0.3

Commit message: Some PCB progress
Parts:
- R18, R19, R20, R21, R22: moved to B.Cu
- moved D1 4.12 mm to (111.3, 87.0)
- moved D2 4.12 mm to (111.3, 91.0)
- moved D3 4.12 mm to (111.3, 95.0)
- moved D4 4.12 mm to (111.3, 99.0)
- moved D5 4.12 mm to (111.3, 103.0)
- moved R13 3.50 mm to (62.0, 79.7), turned to 90 degrees
- moved R14 3.08 mm to (58.5, 79.7), turned to 90 degrees
- moved R18 2.51 mm to (111.3, 87.0), turned to 0 degrees
- moved R19 2.51 mm to (111.3, 91.0), turned to 0 degrees
- moved R20 2.51 mm to (111.3, 95.0), turned to 0 degrees
- moved R21 2.51 mm to (111.3, 99.0), turned to 0 degrees
- moved R22 2.51 mm to (111.3, 103.0), turned to 0 degrees
- moved R6 1.00 mm to (63.0, 126.7)
- moved R12 0.68 mm to (74.8, 126.7)
- moved R15 0.68 mm to (78.8, 126.7), turned to 90 degrees
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Routing:
- net /GI_OUT_0: track 51.6 -> 154.6 mm, vias 0 -> 1
- net +12V: track 127.3 -> 229.1 mm
- net /GI_OUT_1: track 37.2 -> 134.1 mm, vias 0 -> 1
- net /GI_OUT_3: track 55.6 -> 145.9 mm
- net /GI_OUT_2: track 27.1 -> 115.4 mm, vias 0 -> 1
- net /GI_OUT_4: track 98.3 -> 150.9 mm
- net /P4: track 0.00 -> 27.5 mm
- net /P3: track 0.00 -> 21.6 mm
- net Net-(D5-Pad2): track 0.00 -> 6.26 mm, vias 0 -> 1
- net Net-(D4-Pad2): track 0.00 -> 4.60 mm, vias 0 -> 1
- net Net-(D3-Pad2): track 0.00 -> 4.60 mm, vias 0 -> 1
- net Net-(D2-Pad2): track 0.00 -> 4.60 mm, vias 0 -> 1
- net Net-(D1-Pad2): track 0.00 -> 4.60 mm, vias 0 -> 1
Other:
- net class 12V: via_dia 2 -> 0.8; via_drill 1 -> 0.4

Commit message: Some PCB progress
Parts:
- moved R10 53.5 mm to (70.5, 53.9), turned to 90 degrees
- moved R11 53.4 mm to (73.0, 53.9), turned to 90 degrees
- moved R4 48.7 mm to (91.5, 53.9), turned to 90 degrees
- moved R5 48.4 mm to (94.0, 53.9), turned to 90 degrees
- moved R7 48.1 mm to (77.5, 53.9), turned to 90 degrees
- moved R8 47.9 mm to (80.0, 53.9), turned to 90 degrees
- moved R16 30.5 mm to (84.5, 53.9)
- moved R17 30.1 mm to (87.0, 53.9)
- moved R14 26.9 mm to (66.0, 53.9)
- moved R13 25.8 mm to (63.5, 53.9)
- moved R23 21.3 mm to (69.3, 28.5)
- moved R24 20.9 mm to (74.8, 28.5)
- moved RV1 12.1 mm to (84.0, 28.0)
- moved R1 7.82 mm to (79.5, 35.9)
- moved R2 7.82 mm to (82.5, 35.9)
Routing:
- net Net-(Q1-Pad1): track 0.00 -> 65.0 mm
- net Net-(Q3-Pad1): track 0.00 -> 63.5 mm
- net Net-(Q2-Pad1): track 0.00 -> 61.2 mm
- net /5V: track 6.75 -> 57.5 mm
- net GND: track 213.5 -> 263.4 mm, vias 0 -> 4
- net Net-(Q5-Pad1): track 0.00 -> 42.3 mm, vias 0 -> 1
- net Net-(Q4-Pad1): track 0.00 -> 36.0 mm, vias 0 -> 1
- net /P4: track 27.5 -> 9.77 mm
- net /P3: track 21.6 -> 6.01 mm
- net /P0: track 0.00 -> 14.2 mm
- net /P1: track 0.00 -> 10.4 mm
- net /P2: track 0.00 -> 6.82 mm
- net /ZC: track 40.8 -> 42.1 mm

Commit message: Some PCB progress
Parts:
- added ?: MountingHole_4.3mm_M4_DIN965, Mounting_Holes:MountingHole_4.3mm_M4_DIN965, F.Cu at (119.0, 140.5)
- added FLAKIE: , FLAKIE:FLAKIE_inv, F.Cu at (92.5, 34.5)
- added REF**: MountingHole_4.3mm_M4_DIN965, Mounting_Holes:MountingHole_4.3mm_M4_DIN965, F.Cu at (54.0, 139.0)
- added REF**: MountingHole_4.3mm_M4_DIN965, Mounting_Holes:MountingHole_4.3mm_M4_DIN965, F.Cu at (54.5, 31.0)
- added REF**: MountingHole_4.3mm_M4_DIN965, Mounting_Holes:MountingHole_4.3mm_M4_DIN965, F.Cu at (116.0, 32.0)
- C3, R23, R24, U1: moved to B.Cu
- RV1: footprint Potentiometers:Potentiometer_Trimmer_Piher_PT-6v_Horizontal -> Potentiometers:Potentiometer_Trimmer_Piher_PT-10v10_Horizontal_Px10.0mm_Py5.0mm
- moved RV1 16.2 mm to (86.5, 44.0), turned to 90 degrees
- moved R1 14.6 mm to (78.0, 21.4)
- moved R2 14.6 mm to (81.0, 21.4)
- moved R23 14.1 mm to (72.0, 42.4), turned to 270 degrees
- moved R24 13.9 mm to (75.0, 42.4), turned to 90 degrees
- moved C3 13.4 mm to (74.8, 37.0), turned to 0 degrees
- moved U1 0.35 mm to (97.2, 38.7), turned to 180 degrees
Routing:
- net GND: track 263.4 -> 370.7 mm, vias 4 -> 6
- net Net-(A1-Pad20): track 0.00 -> 70.4 mm, vias 0 -> 1
- net /5V: track 57.5 -> 117.4 mm
- net Net-(A1-Pad19): track 0.00 -> 37.4 mm, vias 0 -> 1
- net /T4: track 0.00 -> 36.6 mm, vias 0 -> 1
- net /T3: track 0.00 -> 36.5 mm, vias 0 -> 2
- net /TRIAC: track 23.1 -> 56.0 mm
- net +12V: track 229.1 -> 255.0 mm
- net /T2: track 0.00 -> 24.3 mm, vias 0 -> 1
- net /T0: track 0.00 -> 23.0 mm, vias 0 -> 1
- net /T1: track 0.00 -> 22.0 mm, vias 0 -> 1
- net /D5: track 20.1 -> 32.9 mm, vias 1 -> 0
- net /D7: track 37.4 -> 49.3 mm
- net /D6: track 29.8 -> 39.6 mm, vias 1 -> 0
- net /D4: track 16.7 -> 26.6 mm, vias 1 -> 0
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Other:
- board size 64 x 110 mm -> 64 x 113 mm
- net class Default: clearance 0.3 -> 0.25; trace_width 0.5 -> 0.3
- rule trace_clearance: 0.3 -> 0.25

Commit message: First PCB draft complete
Parts:
- added afterglow: , afterglow:afterglow, F.Cu at (55.5, 109.5)
- R1, R2: moved to B.Cu
- moved R2 67.1 mm to (110.7, 81.5), turned to 180 degrees
- moved R1 21.2 mm to (97.2, 30.5), turned to 180 degrees
- moved ? 3.64 mm to (115.5, 141.5)
- moved REF** 2.55 mm to (54.5, 141.5)
- moved REF** 1.12 mm to (115.5, 31.0)
- moved C3 1.00 mm to (74.8, 38.0)
Routing:
- net /5V: track 117.4 -> 152.7 mm, vias 0 -> 1
- net /TRIAC: track 56.0 -> 76.4 mm
- net GND: track 370.7 -> 387.3 mm
- net /BLANK: track 17.1 -> 21.5 mm
- net /D7: track 49.3 -> 53.6 mm
Other:
- board size 64 x 113 mm -> 69 x 118.5 mm
- board text added: "(c) 2019 by morbid cornflakes"
- board text added: "GI"
- board text added: "v1.0"
