File: afterglow_gi_nano/afterglow_gi_nano.kicad_pcb (KiCad board)
At the start: 2 copper layers, 69 x 118.5 mm, 58 parts, among them J1 Conn_02x17_Odd_Even, J2 POWER_CONN, J3 GI_WPC_J120, J4 GI_WPC_J121, J5 GI_CONN_J119, Q1 FQP30N06L, Q2 FQP30N06L, Q3 FQP30N06L, Q4 FQP30N06L, Q5 FQP30N06L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

Commit message: First PCB draft complete
Parts:
- J119 OUT: renamed from J5
- J120 OUT: renamed from J3
- J121 OUT: renamed from J4
- renumbered REF** to ?
Other:
- board text added: "-12V+"
