File: afterglow_gi_nano/afterglow_gi_nano.sch (KiCad schematic (older format))
At the start: 16 parts

Commit message: Schematic progress
Parts:
- added D2, D3, D4, D5: LED, symbol Device:LED
- added D6: D, symbol Device:D
- added F2, F3, F4, F5: Fuse, symbol Device:Fuse
- added Q2, Q3, Q4, Q5: FQP30N06L, digikey-footprints:TO-220-3, symbol dk_Transistors-FETs-MOSFETs-Single:FQP30N06L
- added R10, R13, R16, R21, R22, R4, R7: 220, symbol Device:R
- added R11, R12, R14, R15, R17, R3, R5, R6, R8, R9: 10k, symbol Device:R
- added R18, R19, R20: 180, symbol Device:R
- added R2: 1.5k, symbol Device:R
- added R23: 1M, symbol Device:R
- added R24: 300k, symbol Device:R
- J2: renamed from J?; value Conn_01x02_Female -> POWER_CONN
- J3: renamed from J?; value Conn_01x11_Male -> GI_WPC_J120
- J4: renamed from J?; value Conn_01x11_Male -> GI_WPC_J121
- J5: renamed from J?; value Conn_01x03_Male -> GI_CONN_J119
- R1: renamed from R?; value R -> 10k
- gave numbers to parts that had none: 11
Connections:
- net +12V: now also F1.2, D6.1 (K), F2.2, F3.2, F4.2, F5.2, R12.2, R15.2, R18.1, R19.1, R20.1, R21.1, R22.1, R23.1, R3.2, R6.2, R9.2; no longer J2.2 (Pin_2)
- net 5V: now also R1.2, R2.2
- net GND: now also J1.14 (Pin_14), J1.16 (Pin_16), J1.18 (Pin_18), J1.20 (Pin_20), J1.22 (Pin_22), J1.24 (Pin_24), J1.26 (Pin_26), J1.28 (Pin_28), J1.30 (Pin_30), Q1.3 (S), U1.10 (GND), Q2.3 (S), Q3.3 (S), Q4.3 (S), Q5.3 (S), R11.1, R14.1, R17.1, R24.2, R5.1, R8.1
- net ZC: now reaches A1.10 (D7)
- net ZC: now also J1.34 (Pin_34)
- net T3: now reaches A1.11 (D8)
- net T3: now also U1.9 (O3)
- net P1: now reaches A1.12 (D9)
- net P1: now also R7.2, R8.2
- net P2: now reaches A1.13 (D10)
- net P2: now also R10.2, R11.2
- net P3: now reaches A1.14 (D11)
- net P3: now also R13.2, R14.2
- net T4: now reaches A1.15 (D12)
- net T4: now also U1.12 (O4)
- net at A1.19 (A0): now also R23.2, R24.1
- net T0: now reaches A1.5 (D2)
- net T0: now also U1.2 (O0)
- net T1: now reaches A1.6 (D3)
- net T1: now also U1.5 (O1)
- net T2: now reaches A1.7 (D4)
- net T2: now also U1.6 (O2)
- net P0: now reaches A1.8 (D5)
- net P0: now also R4.2, R5.2
- net P4: now reaches A1.9 (D6)
- net P4: now also R16.2, R17.2
- net BLANK: now reaches U1.1 (OE)
- net BLANK: now also J1.31 (Pin_31), R1.1
- net TRIAC: now reaches U1.11 (Cp)
- net TRIAC: now also J1.13 (Pin_13), R2.1
- net D4: now reaches U1.13 (D4)
- net D4: now also J1.21 (Pin_21)
- net D5: now reaches U1.14 (D5)
- net D5: now also J1.19 (Pin_19)
- net D6: now reaches U1.17 (D6)
- net D6: now also J1.17 (Pin_17)
- net D7: now reaches U1.18 (D7)
- net D7: now also J1.15 (Pin_15)
- net D0: now reaches U1.3 (D0)
- net D0: now also J1.29 (Pin_29)
- net D1: now reaches U1.4 (D1)
- net D1: now also J1.27 (Pin_27)
- net D2: now reaches U1.7 (D2)
- net D2: now also J1.25 (Pin_25)
- net D3: now reaches U1.8 (D3)
- net D3: now also J1.23 (Pin_23)
- net at Q1.1 (G): now also R4.1
- net GI_OUT_0: now reaches Q1.2 (D)
- net GI_OUT_0: now also D1.1 (K), J3.1 (Pin_1), J4.1 (Pin_1), R3.1
- net at J3.10 (Pin_10): now also J4.10 (Pin_10), F2.1
- net at J3.11 (Pin_11): now also F1.1, J4.11 (Pin_11), J5.3 (Pin_3)
- net GI_OUT_1: now reaches J3.2 (Pin_2)
- net GI_OUT_1: now also J4.2 (Pin_2), D2.1 (K), Q2.2 (D), R6.1
- net GI_OUT_2: now reaches J3.3 (Pin_3)
- net GI_OUT_2: now also J4.3 (Pin_3), D3.1 (K), Q3.2 (D), R9.1
- net GI_OUT_3: now reaches J3.5 (Pin_5)
- net GI_OUT_3: now also J4.5 (Pin_5), D4.1 (K), Q4.2 (D), R12.1
- net GI_OUT_4: now reaches J3.6 (Pin_6)
- net GI_OUT_4: now also J4.6 (Pin_6), J5.1 (Pin_1), D5.1 (K), Q5.2 (D), R15.1
- net at J3.7 (Pin_7): now also J4.7 (Pin_7), F5.1
- net at J3.8 (Pin_8): now also J4.8 (Pin_8), F4.1
- net at J3.9 (Pin_9): now also J4.9 (Pin_9), F3.1
- net at D1.2 (A): now also R18.2
- new net: D6.2 (A), J2.2 (Pin_2)
- new net: D2.2 (A), R19.2
- new net: D3.2 (A), R20.2
- new net: D4.2 (A), R21.2
- new net: D5.2 (A), R22.2
- new net: Q2.1 (G), R7.1
- new net: Q3.1 (G), R10.1
- new net: Q4.1 (G), R13.1
- new net: Q5.1 (G), R16.1
- no-connect marks 13 -> 34
Other:
- note added: "WPC PPD GI OUTPUT"
- note added: "WPC PPD TRIAC INPUT"
- moved on the sheet: A1, C1, C2, C3, D1, F1, J1, J2, J3, J4, J5, Q1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

Commit message: Schematic progressing
Parts:
- removed C2: CP_Small, symbol Device:CP_Small
- added C2: 0.33u, Capacitors_SMD:C_0805_HandSoldering, symbol Device:C_Small
- added J6: Conn_02x17_Odd_Even, Pin_Headers:Pin_Header_Straight_2x17_Pitch2.54mm, symbol Connector_Generic:Conn_02x17_Odd_Even
- C1: footprint (none) -> Capacitors_SMD:C_0805_HandSoldering
- C3: value C_Small -> 0.1u; footprint (none) -> Capacitors_SMD:C_0805_HandSoldering
- D1, D2, D3, D4, D5: footprint (none) -> LEDs:LED_0805_HandSoldering
- D6: footprint (none) -> Diodes_THT:D_5W_P10.16mm_Horizontal
- F1, F2, F3, F4, F5: footprint (none) -> Fuse_Holders_and_Fuses:Fuseholder5x20_horiz_open_lateral_Type-II
- J1: footprint (none) -> Connectors:IDC_Header_Straight_34pins
- J2: footprint (none) -> Connectors_Molex:Molex_KK-41791-02_02x3.96mm_Straight
- J3, J4: footprint (none) -> Connectors_Molex:Molex_KK-41791-11_10x3.96mm_Straight
- J5: footprint (none) -> Connectors_Molex:Molex_KK-41791-03_03x3.96mm_Straight
- Q1, Q2, Q3, Q4, Q5: footprint digikey-footprints:TO-220-3 -> TO_SOT_Packages_THT:TO-220_Vertical
- R1, R10, R11, R12, R13, R14, R15, R16, R17, R18, R19, R2, R20, R21, R22, R23, R24, R3, R4, R5, R6, R7, R8, R9: footprint (none) -> Resistors_SMD:R_0805_HandSoldering
- RV1: footprint (none) -> Potentiometers:Potentiometer_Trimmer_Piher_PT-6v_Horizontal
- U1: footprint (none) -> Housings_DIP:DIP-20_W7.62mm_LongPads
- U2: footprint (none) -> TO_SOT_Packages_THT:TO-220_Vertical
Connections:
- net +12V: now also C2.1
- net BLANK: now also J6.31 (Pin_31)
- net D0: now also J6.29 (Pin_29)
- net D1: now also J6.27 (Pin_27)
- net D2: now also J6.25 (Pin_25)
- net D3: now also J6.23 (Pin_23)
- net D4: now also J6.21 (Pin_21)
- net D5: now also J6.19 (Pin_19)
- net D6: now also J6.17 (Pin_17)
- net D7: now also J6.15 (Pin_15)
- net GND: now also C2.2, J6.14 (Pin_14), J6.16 (Pin_16), J6.18 (Pin_18), J6.20 (Pin_20), J6.22 (Pin_22), J6.24 (Pin_24), J6.26 (Pin_26), J6.28 (Pin_28), J6.30 (Pin_30)
- net TRIAC: now also J6.13 (Pin_13)
- net ZC: now also J6.34 (Pin_34)
- net PIN1: now reaches J1.1 (Pin_1)
- net PIN1: now also J6.1 (Pin_1)
- net PIN10: now reaches J1.10 (Pin_10)
- net PIN10: now also J6.10 (Pin_10)
- net PIN11: now reaches J1.11 (Pin_11)
- net PIN11: now also J6.11 (Pin_11)
- net PIN12: now reaches J1.12 (Pin_12)
- net PIN12: now also J6.12 (Pin_12)
- net PIN2: now reaches J1.2 (Pin_2)
- net PIN2: now also J6.2 (Pin_2)
- net PIN3: now reaches J1.3 (Pin_3)
- net PIN3: now also J6.3 (Pin_3)
- net PIN32: now reaches J1.32 (Pin_32)
- net PIN32: now also J6.32 (Pin_32)
- net PIN33: now reaches J1.33 (Pin_33)
- net PIN33: now also J6.33 (Pin_33)
- net PIN4: now reaches J1.4 (Pin_4)
- net PIN4: now also J6.4 (Pin_4)
- net PIN5: now reaches J1.5 (Pin_5)
- net PIN5: now also J6.5 (Pin_5)
- net PIN6: now reaches J1.6 (Pin_6)
- net PIN6: now also J6.6 (Pin_6)
- net PIN7: now reaches J1.7 (Pin_7)
- net PIN7: now also J6.7 (Pin_7)
- net PIN8: now reaches J1.8 (Pin_8)
- net PIN8: now also J6.8 (Pin_8)
- net PIN9: now reaches J1.9 (Pin_9)
- net PIN9: now also J6.9 (Pin_9)
- no-connect marks 34 -> 20
Other:
- moved on the sheet: C3, D6, J1, J2, R2, U2

Commit message: Designing the PCB
Parts:
- removed J6: Conn_02x17_Odd_Even, Pin_Headers:Pin_Header_Straight_2x17_Pitch2.54mm, symbol Connector_Generic:Conn_02x17_Odd_Even
- J2: footprint Connectors_Molex:Molex_KK-41791-02_02x3.96mm_Straight -> Connectors_Terminal_Blocks:TerminalBlock_Philmore_TB132_02x5mm_Straight
- U1: footprint Housings_DIP:DIP-20_W7.62mm_LongPads -> Housings_SOIC:SOIC-20W_7.5x12.8mm_Pitch1.27mm
Connections:
- net +12V: now also D6.2 (A), J2.2 (Pin_2); no longer C2.1, D6.1 (K), U2.1 (IN)
- new net: C2.1, D6.1 (K), U2.1 (IN)
Other:
- moved on the sheet: D6
Changed lines of the file:
@@
 F 0 "U1" H 1400 5350 50  0000 C CNN
 F 1 "74LS374" H 1400 5250 50  0000 C CNN
-F 2 "Housings_DIP:DIP-20_W7.62mm_LongPads" H 1750 4400 50  0001 C CNN
+F 2 "Housings_SOIC:SOIC-20W_7.5x12.8mm_Pitch1.27mm" H 1750 4400 50  0001 C CNN
 F 3 "http://www.ti.com/lit/gpn/sn74LS374" H 1750 4400 50  0001 C CNN
 	1    1750 4400
@@
 F 0 "J2" H 3494 1025 50  0000 C CNN
 F 1 "POWER_CONN" H 3700 1100 50  0000 C CNN
-F 2 "Connectors_Molex:Molex_KK-41791-02_02x3.96mm_Straight" H 3600 1350 50  0001 C CNN
+F 2 "Connectors_Terminal_Blocks:TerminalBlock_Philmore_TB132_02x5mm_Straight" H 3600 1350 50  0001 C CNN
 F 3 "~" H 3600 1350 50  0001 C CNN
 	1    3600 1350
@@
 L power:+12V #PWR0104
 U 1 1 5C2FAA66
-P 4250 1000
-F 0 "#PWR0104" H 4250 850 50  0001 C CNN
-F 1 "+12V" H 4265 1173 50  0000 C CNN
-F 2 "" H 4250 1000 50  0001 C CNN
-F 3 "" H 4250 1000 50  0001 C CNN
-	1    4250 1000
+P 3900 1000
+F 0 "#PWR0104" H 3900 850 50  0001 C CNN
+F 1 "+12V" H 3915 1173 50  0000 C CNN
+F 2 "" H 3900 1000 50  0001 C CNN
+F 3 "" H 3900 1000 50  0001 C CNN
+	1    3900 1000
 	1    0    0    -1
 $EndComp
 Wire Wire Line
-	4100 1250 4250 1250
-Connection ~ 4250 1250
-Wire Wire Line
-	4250 1250 4400 1250
-Wire Wire Line
-	4250 1250 4250 1000
+	3900 1250 3900 1000
 Wire Wire Line
 	4250 1350 4250 1750
@@
 Wire Wire Line
 	4400 1400 4400 1250
-Connection ~ 4400 1250
 Wire Wire Line
 	4400 1250 4500 1250
@@
 T4
 Wire Wire Line
-	4400 1250 4400 1100
-Text Label 4400 1100 0    50   ~ 0
+	4000 1250 4000 1100
+Text Label 4000 1100 0    50   ~ 0
 12V
 $Comp
@@
 L Device:D D6
 U 1 1 5C3DDC36
-P 3950 1250
-F 0 "D6" H 3950 1034 50  0000 C CNN
-F 1 "D" H 3950 1125 50  0000 C CNN
-F 2 "Diodes_THT:D_5W_P10.16mm_Horizontal" H 3950 1250 50  0001 C CNN
-F 3 "~" H 3950 1250 50  0001 C CNN
-	1    3950 1250
+P 4250 1250
+F 0 "D6" H 4250 1034 50  0000 C CNN
+F 1 "D" H 4250 1125 50  0000 C CNN
+F 2 "Diodes_THT:D_5W_P10.16mm_Horizontal" H 4250 1250 50  0001 C CNN
+F 3 "~" H 4250 1250 50  0001 C CNN
+	1    4250 1250
 	-1   0    0    1
 $EndComp
@@
 	1    0    0    -1
 $EndComp
-$Comp
-L Connector_Generic:Conn_02x17_Odd_Even J6
-U 1 1 5C44FDE0
-P 3050 2500
-F 0 "J6" H 3100 1475 50  0000 C CNN
-F 1 "Conn_02x17_Odd_Even" H 3100 1566 50  0000 C CNN
-F 2 "Pin_Headers:Pin_Header_Straight_2x17_Pitch2.54mm" H 3050 2500 50  0001 C CNN
-F 3 "~" H 3050 2500 50  0001 C CNN
-	1    3050 2500
-	-1   0    0    1
-$EndComp
-Text Label 3250 1800 0    50   ~ 0
-BLANK
-Text Label 3250 1900 0    50   ~ 0
-D0
-Text Label 3250 2000 0    50   ~ 0
-D1
-Text Label 3250 2100 0    50   ~ 0
-D2
-Text Label 3250 2200 0    50   ~ 0
-D3
-Text Label 3250 2300 0    50   ~ 0
-D4
-Text Label 3250 2400 0    50   ~ 0
-D5
-Text Label 3250 2500 0    50   ~ 0
-D6
-Text Label 3250 2600 0    50   ~ 0
-D7
-Text Label 3250 2700 0    50   ~ 0
-TRIAC
-Text Label 2750 1700 2    50   ~ 0
-ZC
-Wire Wire Line
-	2750 1900 2550 1900
-Wire Wire Line
-	2550 1900 2550 2000
-Wire Wire Line
-	2550 2700 2750 2700
-Connection ~ 2550 2700
-Wire Wire Line
-	2550 2700 2550 2800
-Wire Wire Line
-	2750 2600 2550 2600
-Connection ~ 2550 2600
-Wire Wire Line
-	2550 2600 2550 2700
-Wire Wire Line
-	2550 2500 2750 2500
-Connection ~ 2550 2500
-Wire Wire Line
-	2550 2500 2550 2600
-Wire Wire Line
-	2750 2400 2550 2400
-Connection ~ 2550 2400
-Wire Wire Line
-	2550 2400 2550 2500
-Wire Wire Line
-	2550 2300 2750 2300
-Connection ~ 2550 2300
-Wire Wire Line
-	2550 2300 2550 2400
-Wire Wire Line
-	2750 2200 2550 2200
-Connection ~ 2550 2200
-Wire Wire Line
-	2550 2200 2550 2300
-Wire Wire Line
-	2550 2100 2750 2100
-Connection ~ 2550 2100
-Wire Wire Line
-	2550 2100 2550 2200
-Wire Wire Line
-	2750 2000 2550 2000
-Connection ~ 2550 2000
-Wire Wire Line
-	2550 2000 2550 2100
-$Comp
-L power:GND #PWR01
-U 1 1 5C44FE0B
-P 2550 2800
-F 0 "#PWR01" H 2550 2550 50  0001 C CNN
-F 1 "GND" H 2555 2627 50  0000 C CNN
-F 2 "" H 2550 2800 50  0001 C CNN
-F 3 "" H 2550 2800 50  0001 C CNN
-	1    2550 2800
-	1    0    0    -1
-$EndComp
 Text Label 1250 1150 2    50   ~ 0
 PIN32
@@
 Text Label 1750 1050 0    50   ~ 0
 PIN33
-Text Label 3250 1700 0    50   ~ 0
-PIN33
-Text Label 3250 2800 0    50   ~ 0
-PIN11
-Text Label 3250 2900 0    50   ~ 0
-PIN9
-Text Label 3250 3000 0    50   ~ 0
-PIN7
-Text Label 3250 3100 0    50   ~ 0
-PIN5
-Text Label 3250 3200 0    50   ~ 0
-PIN3
-Text Label 3250 3300 0    50   ~ 0
-PIN1
-Text Label 2750 2800 2    50   ~ 0
-PIN12
-Text Label 2750 1800 2    50   ~ 0
-PIN32
-Text Label 2750 3000 2    50   ~ 0
-PIN8
-Text Label 2750 2900 2    50   ~ 0
-PIN10
-Text Label 2750 3100 2    50   ~ 0
-PIN6
-Text Label 2750 3200 2    50   ~ 0
-PIN4
-Text Label 2750 3300 2    50   ~ 0
-PIN2
+Wire Wire Line
+	3800 1250 3900 1250
+Connection ~ 3900 1250
+Wire Wire Line
+	3900 1250 4000 1250
+Connection ~ 4000 1250
+Connection ~ 4400 1250
+Wire Wire Line
+	4000 1250 4100 1250
 $EndSCHEMATC

Commit message: Some PCB progress
Parts:
- RV1: footprint Potentiometers:Potentiometer_Trimmer_Piher_PT-6v_Horizontal -> Potentiometers:Potentiometer_Trimmer_Piher_PT-10v10_Horizontal_Px10.0mm_Py5.0mm
Changed lines of the file:
@@
 F 0 "RV1" H 5481 3896 50  0000 R CNN
 F 1 "R_POT_TRIM" H 5481 3805 50  0000 R CNN
-F 2 "Potentiometers:Potentiometer_Trimmer_Piher_PT-6v_Horizontal" H 5550 3850 50  0001 C CNN
+F 2 "Potentiometers:Potentiometer_Trimmer_Piher_PT-10v10_Horizontal_Px10.0mm_Py5.0mm" H 5550 3850 50  0001 C CNN
 F 3 "~" H 5550 3850 50  0001 C CNN
 	1    5550 3850
