File: afterglow_gi_nano_ps/_autosave-afterglow_gi_nano_ps.sch (KiCad schematic (older format))
At the start: 64 parts, among them J1 Conn_02x17_Odd_Even, J2 POWER_CONN, J3 GI_WPC_J120, J4 GI_WPC_J121, J5 GI_CONN_J119, J6 Conn_01x12_Male, Q1 FQP30N06L, Q2 FQP30N06L, Q3 FQP30N06L, Q4 FQP30N06L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

Commit message: A PCB layout proposal
Parts:
- J6: footprint Connectors_Molex:Molex_KK-6410-12_12x2.54mm_Straight -> Connectors_Molex:Molex_KK-41791-12_10x3.96mm_Straight
- Q6, Q7, Q8, Q9: footprint digikey-footprints:TO-220-3 -> TO_SOT_Packages_THT:TO-220_Vertical
Changed lines of the file:
@@
 F 0 "Q7" H 7408 2353 60  0000 L CNN
 F 1 "FQP30N06L" H 7408 2247 60  0000 L CNN
-F 2 "digikey-footprints:TO-220-3" H 7500 2500 60  0001 L CNN
+F 2 "TO_SOT_Packages_THT:TO-220_Vertical" H 7500 2500 60  0001 L CNN
 F 3 "https://www.fairchildsemi.com/datasheets/FQ/FQP30N06L.pdf" H 7500 2600 60  0001 L CNN
 F 4 "FQP30N06L-ND" H 7500 2700 60  0001 L CNN "Digi-Key_PN"
@@
 F 0 "J6" H 6008 1981 50  0000 C CNN
 F 1 "Conn_01x12_Male" H 6008 1890 50  0000 C CNN
-F 2 "Connectors_Molex:Molex_KK-6410-12_12x2.54mm_Straight" H 5900 1300 50  0001 C CNN
+F 2 "Connectors_Molex:Molex_KK-41791-12_10x3.96mm_Straight" H 5900 1300 50  0001 C CNN
 F 3 "~" H 5900 1300 50  0001 C CNN
 	1    5900 1300
@@
 F 0 "Q9" H 9258 2353 60  0000 L CNN
 F 1 "FQP30N06L" H 9258 2247 60  0000 L CNN
-F 2 "digikey-footprints:TO-220-3" H 9350 2500 60  0001 L CNN
+F 2 "TO_SOT_Packages_THT:TO-220_Vertical" H 9350 2500 60  0001 L CNN
 F 3 "https://www.fairchildsemi.com/datasheets/FQ/FQP30N06L.pdf" H 9350 2600 60  0001 L CNN
 F 4 "FQP30N06L-ND" H 9350 2700 60  0001 L CNN "Digi-Key_PN"
@@
 F 0 "Q8" H 9258 1503 60  0000 L CNN
 F 1 "FQP30N06L" H 9258 1397 60  0000 L CNN
-F 2 "digikey-footprints:TO-220-3" H 9350 1650 60  0001 L CNN
+F 2 "TO_SOT_Packages_THT:TO-220_Vertical" H 9350 1650 60  0001 L CNN
 F 3 "https://www.fairchildsemi.com/datasheets/FQ/FQP30N06L.pdf" H 9350 1750 60  0001 L CNN
 F 4 "FQP30N06L-ND" H 9350 1850 60  0001 L CNN "Digi-Key_PN"
@@
 F 0 "Q6" H 7058 1853 60  0000 L CNN
 F 1 "FQP30N06L" H 7058 1747 60  0000 L CNN
-F 2 "digikey-footprints:TO-220-3" H 7150 2000 60  0001 L CNN
+F 2 "TO_SOT_Packages_THT:TO-220_Vertical" H 7150 2000 60  0001 L CNN
 F 3 "https://www.fairchildsemi.com/datasheets/FQ/FQP30N06L.pdf" H 7150 2100 60  0001 L CNN
 F 4 "FQP30N06L-ND" H 7150 2200 60  0001 L CNN "Digi-Key_PN"
